Commit message: [fix] moveit demo

File: colcon_ws/src/panda_description/urdf/panda.urdf (robot description, URDF)
Before this commit: robot panda, 12 links, 11 joints
Links:
- link panda_hand: geometry collision mesh filename=file://$(find moveit_resources_panda_description)/meshes/co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; visual mesh filename=file://$(find moveit_resources_panda_description)/meshes/vi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
- link panda_leftfinger: geometry collision mesh filename=file://$(find moveit_resources_panda_description)/meshes/co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; visual mesh filename=file://$(find moveit_resources_panda_description)/meshes/vi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
- link panda_link0: geometry collision mesh filename=file://$(find moveit_resources_panda_description)/meshes/co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; visual mesh filename=file://$(find moveit_resources_panda_description)/meshes/vi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
- link panda_link1: geometry collision mesh filename=file://$(find moveit_resources_panda_description)/meshes/co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; visual mesh filename=file://$(find moveit_resources_panda_description)/meshes/vi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
- link panda_link2: geometry collision mesh filename=file://$(find moveit_resources_panda_description)/meshes/co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; visual mesh filename=file://$(find moveit_resources_panda_description)/meshes/vi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
- link panda_link3: geometry collision mesh filename=file://$(find moveit_resources_panda_description)/meshes/co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; visual mesh filename=file://$(find moveit_resources_panda_description)/meshes/vi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
- link panda_link4: geometry collision mesh filename=file://$(find moveit_resources_panda_description)/meshes/co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; visual mesh filename=file://$(find moveit_resources_panda_description)/meshes/vi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
- link panda_link5: geometry collision mesh filename=file://$(find moveit_resources_panda_description)/meshes/co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; visual mesh filename=file://$(find moveit_resources_panda_description)/meshes/vi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
- link panda_link6: geometry collision mesh filename=file://$(find moveit_resources_panda_description)/meshes/co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; visual mesh filename=file://$(find moveit_resources_panda_description)/meshes/vi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
- link panda_link7: geometry collision mesh filename=file://$(find moveit_resources_panda_description)/meshes/co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; visual mesh filename=file://$(find moveit_resources_panda_description)/meshes/vi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
- link panda_rightfinger: geometry collision mesh filename=file://$(find moveit_resources_panda_description)/meshes/co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; visual mesh filename=file://$(find moveit_resources_panda_description)/meshes/vi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
